Commit message: model is existing peacefully with everything in the correct place

File: src/fanipulator/urdf/fanipulator.urdf (robot description, URDF)
Before this commit: robot fanipulator, 14 links, 13 joints
Joints:
- joint joint_wrist_non_motor_support: origin xyz=-0.0365783595746249 0.00525000000000003 0.0415351375358365 rpy=0 0.887232723469578 0 -> xyz=-0.017 0.00925000000000003 0.0175 rpy=0 4.0288227234695 0

Commit message: atleast the gripper is working somewhat correctly

File: src/fanipulator/urdf/fanipulator.urdf (robot description, URDF)
Before this commit: robot fanipulator, 14 links, 13 joints
Joints:
- joint joint_arm01_arm02: limit lower=-.1 upper=.1 effort=0 velocity=0 -> lower=-.1.57 upper=.1.57 effort=0 velocity=0
- joint joint_arm03_wrist: limit lower=-.1 upper=.1 effort=0 velocity=0 -> lower=-.1.57 upper=.1.57 effort=0 velocity=0
- joint joint_motor_gear_finger: limit lower=-.1 upper=.1 effort=0 velocity=0 -> lower=-.1.57 upper=.1.57 effort=0 velocity=0; mimic (none) -> joint=joint_wrist_motor_gear multiplier=-1.0
- joint joint_non_motor_gear_finger: limit lower=-.1 upper=.1 effort=0 velocity=0 -> lower=-.1.57 upper=.1.57 effort=0 velocity=0; mimic (none) -> joint=joint_wrist_motor_gear multiplier=-1.0
- joint joint_waist_arm01: limit lower=-.1 upper=.1 effort=0 velocity=0 -> lower=-.1.57 upper=.1.57 effort=0 velocity=0
- joint joint_wrist_motor_gear: limit lower=-.1 upper=.1 effort=0 velocity=0 -> lower=-.1.57 upper=.1.57 effort=0 velocity=0
- joint joint_wrist_motor_support: limit lower=-.1 upper=.1 effort=0 velocity=0 -> lower=-.1.57 upper=.1.57 effort=0 velocity=0; mimic (none) -> joint=joint_wrist_motor_gear multiplier=1.0
- joint joint_wrist_non_motor_gear: limit lower=-.1 upper=.1 effort=0 velocity=0 -> lower=-.1.57 upper=.1.57 effort=0 velocity=0; mimic (none) -> joint=joint_wrist_motor_gear multiplier=-1.0
- joint joint_wrist_non_motor_support: limit lower=-.1 upper=.1 effort=0 velocity=0 -> lower=-.1.57 upper=.1.57 effort=0 velocity=0; mimic (none) -> joint=joint_wrist_motor_gear multiplier=-1.0

Commit message: everything is working as it should

File: src/fanipulator/urdf/fanipulator.urdf (robot description, URDF)
Before this commit: robot fanipulator, 14 links, 13 joints
Joints:
- joint joint_arm01_arm02: limit lower=-.1.57 upper=.1.57 effort=0 velocity=0 -> lower=-1.57 upper=1.57 effort=0 velocity=0; origin xyz=-0.0064428 0.15415 0.0222 rpy=0 0 1.7573 -> xyz=-0.00 0.12 0.0222 rpy=0 0 1.7573
- joint joint_arm03_wrist: limit lower=-.1.57 upper=.1.57 effort=0 velocity=0 -> lower=-1.57 upper=1.57 effort=0 velocity=0
- joint joint_motor_gear_finger: limit lower=-.1.57 upper=.1.57 effort=0 velocity=0 -> lower=-1.57 upper=1.57 effort=0 velocity=0
- joint joint_non_motor_gear_finger: limit lower=-.1.57 upper=.1.57 effort=0 velocity=0 -> lower=-1.57 upper=1.57 effort=0 velocity=0
- joint joint_waist_arm01: limit lower=-.1.57 upper=.1.57 effort=0 velocity=0 -> lower=-1.57 upper=1.57 effort=0 velocity=0
- joint joint_wrist_motor_gear: limit lower=-.1.57 upper=.1.57 effort=0 velocity=0 -> lower=-1.57 upper=1.57 effort=0 velocity=0
- joint joint_wrist_motor_support: limit lower=-.1.57 upper=.1.57 effort=0 velocity=0 -> lower=-1.57 upper=1.57 effort=0 velocity=0
- joint joint_wrist_non_motor_gear: limit lower=-.1.57 upper=.1.57 effort=0 velocity=0 -> lower=-1.57 upper=1.57 effort=0 velocity=0
- joint joint_wrist_non_motor_support: limit lower=-.1.57 upper=.1.57 effort=0 velocity=0 -> lower=-1.57 upper=1.57 effort=0 velocity=0

File: src/manipulator/urdf/manipulator.urdf (robot description, URDF)
Before this commit: robot manipulator, 13 links, 12 joints
Links:
- removed link link_finger_motor
- removed link link_finger_non_motor
- removed link link_gear_motor
- removed link link_gear_non_motor
- removed link link_gripper_wrist
- removed link link_support_motor
- removed link link_support_non_motor
- added link link_motor_finger, mass 0.00255464599773235; collision mesh filename=package://manipulator/meshes/link_motor_finger.STL; visual mesh filename=package://manipulator/meshes/link_motor_finger.STL
- added link link_motor_gear, mass 0.0025818082333029; collision mesh filename=package://manipulator/meshes/link_motor_gear.STL; visual mesh filename=package://manipulator/meshes/link_motor_gear.STL
- added link link_motor_support, mass 0.000798762413184692; collision mesh filename=package://manipulator/meshes/link_motor_support.STL; visual mesh filename=package://manipulator/meshes/link_motor_support.STL
- added link link_non_motor_finger, mass 0.00255464579636163; collision mesh filename=package://manipulator/meshes/link_non_motor_finger.STL; visual mesh filename=package://manipulator/meshes/link_non_motor_finger.STL
- added link link_non_motor_gear, mass 0.00265818035071168; collision mesh filename=package://manipulator/meshes/link_non_motor_gear.STL; visual mesh filename=package://manipulator/meshes/link_non_motor_gear.STL
- added link link_non_motor_support, mass 0.000798762413184692; collision mesh filename=package://manipulator/meshes/link_non_motor_support.STL; visual mesh filename=package://manipulator/meshes/link_non_motor_support.STL
- added link link_servo, mass 0.00717741212346476; collision mesh filename=package://manipulator/meshes/link_servo.STL; visual mesh filename=package://manipulator/meshes/link_servo.STL
- added link link_wrist, mass 0.0160406157199611; collision mesh filename=package://manipulator/meshes/link_wrist.STL; visual mesh filename=package://manipulator/meshes/link_wrist.STL
- link link_arm01: mass 0.0640544606432968 -> 0.064057051230774
- link link_arm02: mass 0.0470979601767716 -> 0.0470979731232057
- link link_arm03: mass 0.0164704027054544 -> 0.0164703704574985
- link link_waist: mass 0.0736482065125356 -> 0.073648017160832
Joints:
- removed joint joint_arm03_gripper
- removed joint joint_gear_motor_finger
- removed joint joint_gear_motor_support
- removed joint joint_gear_non_motor_finger
- removed joint joint_gear_non_motor_support
- removed joint joint_wrist_gear_motor
- removed joint joint_wrist_gear_non_motor
- added joint joint_arm03_wrist: type revolute, parent link_arm03, child link_wrist, origin xyz=0 0.028 -0.0155 rpy=0 0 2.97515466965945, axis 0 0 -1, limit lower=-1.4 upper=1.4 effort=338 velocity=10
- added joint joint_motor_gear_finger: type continuous, parent link_motor_gear, child link_motor_finger, origin xyz=0.028766 0.010867 0.002 rpy=3.1416 0 0, axis 0 0 -1, limit lower=-1.4 upper=1.4 effort=338 velocity=10, mimic joint=joint_wrist_motor_gear multiplier=-0.8
- added joint joint_non_motor_gear_finger: type revolute, parent link_non_motor_gear, child link_non_motor_finger, origin xyz=0.029123 0.0098705 0.002 rpy=-3.1416 0 1.5482, axis 0 0 -1, limit lower=-1.4 upper=1.4 effort=338 velocity=10, mimic joint=joint_wrist_motor_gear multiplier=-0.8
- added joint joint_wrist_motor_gear: type revolute, parent link_wrist, child link_motor_gear, origin xyz=0.0361395051353438 -0.0200499044528838 0.0189000000000357 rpy=-1.5707963267949 -0.852106499830379 -0.102417256192125, axis 0 0 -1, limit lower=-0.09 upper=0.0275 effort=338 velocity=10
- added joint joint_wrist_motor_support: type revolute, parent link_wrist, child link_motor_support, origin xyz=0.0562391804526159 -0.0201051506339748 0.0100000000000436 rpy=-3.14159265358979 -0.81681166488745 -0.102417256192128, axis 0 1 0, limit lower=-1.4 upper=1.4 effort=338 velocity=10, mimic joint=joint_wrist_motor_gear multiplier=1.2
- added joint joint_wrist_non_motor_gear: type revolute, parent link_wrist, child link_non_motor_gear, origin xyz=0.0361395051353807 -0.0200499044528875 -0.00800000000000281 rpy=1.5707963267949 0.696091483245096 -0.102417256192129, axis 0 0 1, limit lower=-1.4 upper=1.4 effort=338 velocity=10, mimic joint=joint_wrist_motor_gear multiplier=-1.0
- added joint joint_wrist_non_motor_support: type revolute, parent link_wrist, child link_non_motor_support, origin xyz=0.0558302272421884 -0.0240841903763851 0 rpy=-1.5707963267949 -0.852106499830378 -0.102417256192126, axis 0 0 -1, limit lower=-1.4 upper=1.4 effort=338 velocity=10, mimic joint=joint_wrist_motor_gear multiplier=-1.2
- added joint joint_wrist_servo_fixed: type fixed, parent link_wrist, child link_servo, origin xyz=0.0393088925164345 0.010787653550768 0.024 rpy=1.67321358298702 -1.5707963267949 0, axis 0 0 0
- joint joint_arm01_arm02: axis 0 0 1 -> 0 0 -1; limit (none) -> lower=-1.4 upper=1.4 effort=338 velocity=10; origin xyz=0 0.120000000000003 0 rpy=0 0 1.1544064242663 -> xyz=0 0.12 0.015 rpy=3.14159265358979 0 -2.94369460393837; type continuous -> revolute
- joint joint_arm02_arm03: axis 0 1 0 -> 0 -1 0; limit (none) -> lower=-1.4 upper=1.4 effort=338 velocity=10; origin xyz=0.103168801289468 0.00530000000121461 0.00949999999992188 rpy=0 -1.24589601241689 -1.57079632682694 -> xyz=-0.0001165850778517 0.090954594899946 -0.0151145368982072 rpy=3.14159265358979 0.503971856291605 -3.13017769589601
- joint joint_base_dummy: child link_dummy -> base_link; origin xyz=0 0 0 rpy=0 0 0 -> xyz=0 0 0.1 rpy=0.52 0.3 0; parent base_link -> link_dummy
- joint joint_base_waist: limit (none) -> lower=0 upper=0 effort=0 velocity=0; origin xyz=0.100478709174496 -0.0656562967351186 0.0509945925861506 rpy=1.86216248284797 -0.368573868525035 -1.83635830754677 -> xyz=0.104619716257001 -0.0747184271679116 0.0311676085902517 rpy=1.24263440323189 0.336564980145166 1.19877807114456
- joint joint_waist_arm01: limit (none) -> lower=-1.4 upper=1.4 effort=338 velocity=10; origin xyz=0 0.018090375352197 -0.0139100000000071 rpy=1.5707963267946 1.10898105062242 1.57079632679463 -> xyz=-0.0182 0.0402799999999999 -0.0139099999999999 rpy=1.57079632679491 1.44053245288332 1.57079632679491; type continuous -> revolute
