Commit message: just before changing values stupidly

File: src/manipulator/urdf/manipulator.urdf (robot description, URDF)
Before this commit: robot manipulator, 12 links, 11 joints
Links:
- added link link_dummy; visual box size=0.01 0.01 0.01
Joints:
- added joint joint_base_dummy: type fixed, parent base_link, child link_dummy, origin xyz=0 0 0 rpy=0 0 0

Commit message: added transmission and gazebo tags, don't know if they are correct

File: src/manipulator/urdf/manipulator.urdf (robot description, URDF)
Before this commit: robot manipulator, 14 links, 13 joints
Links:
- removed link link_dummy
- added link world; visual box size=0.01 0.01 0.01
Joints:
- removed joint joint_base_dummy
- added joint joint_world_base_link: type fixed, parent world, child base_link, origin xyz=0 0 0.1 rpy=0.52 0.3 0
- joint joint_base_waist: limit lower=0 upper=0 effort=0 velocity=0 -> lower=0 upper=0 effort=338 velocity=10
- joint joint_motor_gear_finger: limit lower=-1.4 upper=1.4 effort=338 velocity=10 -> lower=-1.4 upper=1.4 effort=0 velocity=10
- joint joint_non_motor_gear_finger: limit lower=-1.4 upper=1.4 effort=338 velocity=10 -> lower=-1.4 upper=1.4 effort=0 velocity=10
- joint joint_wrist_motor_support: limit lower=-1.4 upper=1.4 effort=338 velocity=10 -> lower=-1.4 upper=1.4 effort=0 velocity=10
- joint joint_wrist_non_motor_gear: limit lower=-1.4 upper=1.4 effort=338 velocity=10 -> lower=-1.4 upper=1.4 effort=0 velocity=10
- joint joint_wrist_non_motor_support: limit lower=-1.4 upper=1.4 effort=338 velocity=10 -> lower=-1.4 upper=1.4 effort=0 velocity=10

Commit message: final commit

File: src/manipulator/urdf/manipulator.urdf (robot description, URDF)
Before this commit: robot manipulator, 14 links, 13 joints
Joints:
- joint joint_world_base_link: origin xyz=0 0 0.1 rpy=0.52 0.3 0 -> xyz=0 0 0.2 rpy=0.52 0.3 0
